File: hardware/scu-devkitv1/scu-devkitv1.kicad_sch (KiCad schematic)
At the start: 4 parts

Commit message: HARDWARE FINISHED
Parts:
- added D2: D, scu-Library:schottky, symbol Device:D
- added D3: LED, LED_THT:LED_D3.0mm_Clear, symbol Device:LED
- added J1: Conn_01x04_Female, TerminalBlock_Altech:Altech_AK300_1x04_P5.00mm_45-Degree, symbol Connector:Conn_01x04_Female
- added R1: 120ohms, Resistor_THT:R_Axial_DIN0207_L6.3mm_D2.5mm_P10.16mm_Horizontal, symbol Device:R_US
- added U2: MicroSD, scu-Library:SCU_SD_mini, symbol scu2021:Baja_SD
- added U5: GPRS_-_SIM800L, scu-Library:GPRS - SIM800L, symbol SCU_components:GPRS_-_SIM800L
- added U6: MCP2515-SHIELD, scu-Library:MCP2515-SHIELD, symbol scu-library:MCP2515-SHIELD
- D1: renamed from D?; footprint custom_library:schottky -> scu-Library:schottky
- U3, U4: renamed from U?; footprint custom_library:LM2596 MINI 360 -> scu-Library:LM2596 MINI 360
- gave numbers to parts that had none: 1
Connections:
- net 12V: now also D2.2 (A), J1.1 (Pin_1)
- net 4V: now also U5.2 (VCC)
- net 5V: now also U6.7 (VCC)
- net Earth: now also D3.1 (K), J1.4 (Pin_4), U2.6 (GND), U5.6 (GND), U6.6 (GND)
- net VBAT+: now also D2.1 (K)
- net 3V3: now reaches U1.16 (3V3)
- net 3V3: now also U2.5 (VCC)
- net DEBUG LED 2: now reaches U1.18 (IO15)
- net DEBUG LED 2: now also R1.1
- net CAN_CS: now reaches U1.20 (IO4)
- net CAN_CS: now also U6.5 (CS)
- net GPRS RX: now reaches U1.21 (IO16)
- net GPRS RX: now also U5.4 (RXD)
- net GPRS TX: now reaches U1.22 (IO17)
- net GPRS TX: now also U5.5 (TXD)
- net CS: now reaches U1.23 (IO5)
- net CS: now also U2.1 (CS)
- net SCK: now reaches U1.24 (IO18)
- net SCK: now also U2.2 (SCK), U6.2 (SCK)
- net MISO: now reaches U1.25 (IO19)
- net MISO: now also U2.4 (MISO), U6.4 (SO)
- net MOSI: now reaches U1.30 (IO23)
- net MOSI: now also U2.3 (MOSI), U6.3 (SI)
- new net: D3.2 (A), R1.2
- new net CAN_HIGH: J1.2 (Pin_2), U6.8 (CAN_HIGH)
- new net CAN_INT: U6.1 (INT)
- new net CAN_LOW: J1.3 (Pin_3), U6.9 (CAN_LOW)
Other:
- note added: "CAN SHIELD"
- note added: "Debugging LEDs"
- note added: "Embbeded input"
- note added: "GPRS Module"
- note added: "SD Module"
